Commit message: Working CA1, working on CA2

File: src/rb2301_description/urdf/nanocar_description.urdf (robot description, URDF)
Before this commit: robot NanoCar, 9 links, 8 joints
Links:
- link back_left_wheel_link: geometry collision mesh filename=package://rb2301_description/meshes/nanocar/back_left_wheel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; visual mesh filename=package://rb2301_description/meshes/nanocar/back_left_wheel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
- link back_right_wheel_link: geometry collision mesh filename=package://rb2301_description/meshes/nanocar/back_right_whee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; visual mesh filename=package://rb2301_description/meshes/nanocar/back_right_whee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
- link base_camera_link: geometry collision mesh filename=package://rb2301_description/meshes/nanocar/base_camera_lin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; visual mesh filename=package://rb2301_description/meshes/nanocar/base_camera_lin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
- link base_laser_link: geometry collision mesh filename=package://rb2301_description/meshes/nanocar/base_laser_link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; visual mesh filename=package://rb2301_description/meshes/nanocar/base_laser_link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
- link base_link: geometry collision mesh filename=package://rb2301_description/meshes/nanocar/base_link.STL; visual mesh filename=package://rb2301_description/meshes/nanocar/base_link.STL
- link front_left_wheel_link: geometry collision mesh filename=package://rb2301_description/meshes/nanocar/front_left_whee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; visual mesh filename=package://rb2301_description/meshes/nanocar/front_left_whee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
- link front_right_wheel_link: geometry collision mesh filename=package://rb2301_description/meshes/nanocar/front_right_whe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; visual mesh filename=package://rb2301_description/meshes/nanocar/front_right_whe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
- link imu_link: geometry collision mesh filename=package://rb2301_description/meshes/nanocar/imu.STL; visual mesh filename=package://rb2301_description/meshes/nanocar/imu.STL
